File: pcb/fin-ltm.kicad_pcb (KiCad board)
At the start: 2 copper layers, 112.5 x 109.8 mm, 167 parts, among them J1 Connector, USB-TYPE-C-16P, J2 Test Connector, Q1 MMBT3904, Q2 HL3415A, U1 ESP32-C3FH4, U2 RT9080, U3 SN74LV1T34DBV, X1 40MHz, 15pF

Commit message: pcb
Parts:
- moved J2 97.7 mm to (22.5, 59.0)
- moved C1 5.49 mm to (24.5, 37.0)
- moved R6 4.12 mm to (27.5, 37.0)
- moved D4 2.90 mm to (21.6, 36.8)
- moved C19 2.83 mm to (26.5, 37.0), turned to -90 degrees
- moved R5 2.55 mm to (34.0, 38.0), turned to -90 degrees
- moved F1 2.16 mm to (21.6, 41.8), turned to 180 degrees
- moved C13 2.00 mm to (25.5, 37.0)
- moved U2 1.61 mm to (20.8, 31.9)
- moved C2 1.50 mm to (20.2, 34.5)
- moved Q1 1.10 mm to (29.7, 39.9)
- moved C12 1.00 mm to (33.0, 38.0)
- moved R4 1.00 mm to (32.0, 38.0)
- moved D2 0.35 mm to (21.6, 39.2), turned to 180 degrees
- moved Q2 0.05 mm to (26.3, 39.9), turned to -90 degrees
Connections:
- R18 pad 2: /DISPLAY_SCL -> /DISPLAY_SDA
- R19 pad 2: /DISPLAY_SDA -> /DISPLAY_SCL
- U1 pad 4: /DISPLAY_SCL -> /DISPLAY_SDA
- U1 pad 5: /DISPLAY_SDA -> /DISPLAY_SCL
Routing:
- net /BRIGHTNESS_DOWN_BUTTON: track 7.78 -> 127.6 mm
- net /BRIGHTNESS_UP_BUTTON: track 10.0 -> 129.6 mm
- net /POWER_BUTTON: track 13.9 -> 128.7 mm, vias 1 -> 3
- net Net-(C1-Pad2): track 222.5 -> 141.2 mm, vias 6 -> 8
- net /DISPLAY_SCL: track 16.2 -> 85.5 mm, vias 1 -> 3
- net /DISPLAY_SDA: track 16.2 -> 78.8 mm, vias 1 -> 3
- net +3V3: track 189.3 -> 226.8 mm
- net /MCU_TX: track 3.06 -> 34.0 mm, vias 1 -> 3
- net /Leds/LED_DATA_5V: track 35.2 -> 5.33 mm, vias 3 -> 1
- net /MCU_RX: track 5.98 -> 31.9 mm, vias 1 -> 3
- net +5V: track 6.53 -> 31.2 mm, vias 1 -> 3
- net /Reset: track 17.9 -> 40.9 mm, vias 1 -> 3
- net VBUS: track 174.3 -> 164.5 mm, vias 6 -> 8
- net /LED_POWER_CTRL: track 10.9 -> 12.8 mm
- net Net-(Q1-C): track 6.48 -> 4.89 mm
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
Commit message: pcb 2
Parts:
- moved D191 31.8 mm to (94.8, 46.5)
- moved S3 30.2 mm to (120.2, 91.0)
- moved D152 29.6 mm to (81.8, 49.0)
- moved D151 29.4 mm to (81.8, 46.5)
- moved D113 27.8 mm to (68.0, 51.5)
- moved D112 27.6 mm to (68.0, 49.0)
- moved D111 27.5 mm to (68.0, 46.5)
- moved D140 24.8 mm to (75.0, 69.0)
- moved D1 24.8 mm to (120.2, 62.2)
- moved D10 24.8 mm to (120.2, 73.8)
- moved D5 24.8 mm to (120.2, 64.2)
- moved D7 24.8 mm to (120.2, 70.0)
- moved D8 24.8 mm to (120.2, 68.0)
- moved D9 24.8 mm to (120.2, 75.8)
- moved R12 24.8 mm to (122.5, 70.0)
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Connections:
- R16 pad 2: /BRIGHTNESS_UP_BUTTON -> /BRIGHTNESS_DOWN_BUTTON
- R17 pad 2: /BRIGHTNESS_DOWN_BUTTON -> /BRIGHTNESS_UP_BUTTON
- U1 pad 15: /BRIGHTNESS_UP_BUTTON -> /BRIGHTNESS_DOWN_BUTTON
- U1 pad 16: /BRIGHTNESS_DOWN_BUTTON -> /BRIGHTNESS_UP_BUTTON
Routing:
- net /MODE_BUTTON: track 2.19 -> 170.4 mm, vias 1 -> 4
- net Net-(C1-Pad2): track 141.2 -> 203.9 mm, vias 8 -> 9
- net /Leds/LED_DATA_5V: track 5.33 -> 49.1 mm, vias 1 -> 3
- net +5V: track 31.2 -> 62.4 mm, vias 3 -> 5
- net /SERVER_LED: track 149.1 -> 124.1 mm
- net /WIFI_LED: track 141.8 -> 116.9 mm
- net /BRIGHTNESS_DOWN_BUTTON: track 127.6 -> 148.9 mm, vias 1 -> 2
- net +3V3: track 226.8 -> 210.5 mm
- net /POWER_BUTTON: track 128.7 -> 144.9 mm, vias 3 -> 4
- net /DISPLAY_SDA: track 78.8 -> 92.6 mm
- net /BRIGHTNESS_UP_BUTTON: track 129.6 -> 140.8 mm, vias 1 -> 2
- net /MCU_RX: track 31.9 -> 41.1 mm
- net VBUS: track 164.5 -> 156.0 mm
- net /MCU_TX: track 34.0 -> 42.5 mm
- net /DISPLAY_SCL: track 85.5 -> 93.2 mm
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Other:
- board text added: "OLED here?"
- board text added: "Reroute 5V and LED_DATA traces if needed"
