File: pcb/fin-ltm.kicad_pcb (KiCad board)
At the start: 2 copper layers, 112.5 x 109.8 mm, 167 parts, among them J1 Connector, USB-TYPE-C-16P, J2 Test Connector, Q1 MMBT3904, Q2 HL3415A, U1 ESP32-C3FH4, U2 RT9080, U3 SN74LV1T34DBV, X1 40MHz, 15pF

Commit message: pcb tweaks
Parts:
- moved S4 12.0 mm to (120.2, 97.2)
- moved S1 6.00 mm to (120.2, 103.2)
- moved S2 6.00 mm to (120.2, 109.2)
Routing:
- net VBUS: track 156.0 -> 135.1 mm
- net Net-(C1-Pad2): track 203.9 -> 186.9 mm
- net /MODE_BUTTON: track 170.4 -> 158.5 mm
- net /BRIGHTNESS_DOWN_BUTTON: track 148.9 -> 154.6 mm
- net /BRIGHTNESS_UP_BUTTON: track 140.8 -> 146.5 mm
- net /Leds/LED_DATA_5V: track 49.1 -> 44.7 mm
- net +5V: track 62.4 -> 59.5 mm
- net /POWER_BUTTON: track 144.9 -> 145.6 mm
- net /MCU_TX: track 42.5 -> 43.1 mm

Commit message: add oled
Parts:
- added J3: Display, Custom:OLED_1306_THT_pinheader, F.Cu at (108.9, 43.8)
- AE1: footprint Library:Inverted_F_Antenna_2.4Ghz_1.0mmPCB_TI_CC2430DB.pretty -> Custom:Inverted_F_Antenna_2.4Ghz_1.0mmPCB_TI_CC2430DB.pretty
- J2: footprint Library:Test_connector -> Custom:Test_connector
- moved C22 7.76 mm to (105.1, 41.5), turned to 180 degrees
- moved D101 5.71 mm to (60.8, 50.8)
- moved D102 5.71 mm to (60.8, 53.3)
- moved D103 5.71 mm to (60.8, 55.8)
- moved D104 5.71 mm to (60.8, 58.3)
- moved D105 5.71 mm to (60.8, 60.8)
- moved D106 5.71 mm to (60.8, 63.3)
- moved D107 5.71 mm to (60.8, 65.8)
- moved D108 5.71 mm to (60.8, 68.3)
- moved D109 5.71 mm to (60.8, 70.8)
- moved D110 5.71 mm to (60.8, 73.3)
- moved D111 5.71 mm to (64.2, 50.8)
- moved D112 5.71 mm to (64.2, 53.3)
- moved D113 5.71 mm to (64.2, 55.8)
- moved D114 5.71 mm to (64.2, 58.3)
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Connections:
- C22 pad 1: VBUS -> +3V3
Routing:
- net +3V3: track 210.8 -> 238.5 mm, vias 10 -> 11
- net Net-(C1-Pad2): track 186.9 -> 202.8 mm
- net VBUS: track 135.1 -> 148.0 mm
- net /DISPLAY_SDA: track 92.8 -> 100.8 mm
- net /DISPLAY_SCL: track 93.5 -> 98.1 mm
- net /SERVER_LED: track 124.1 -> 121.5 mm
- net /WIFI_LED: track 116.9 -> 114.2 mm
- net /BRIGHTNESS_DOWN_BUTTON: track 154.6 -> 151.9 mm
- net /BRIGHTNESS_UP_BUTTON: track 146.5 -> 143.8 mm
- net /POWER_BUTTON: track 145.6 -> 143.0 mm
- net /MODE_BUTTON: track 158.5 -> 156.0 mm
- net +5V: track 59.5 -> 58.0 mm
- net /Leds/LED_DATA_5V: track 44.7 -> 43.2 mm
- net GND: vias 57 -> 55
Other:
- board text added: "This might be the wrong footprint (maybe not)"
- board text removed: "OLED here?"

Commit message: led routing
Parts:
- removed C22: 10uF, PCM_JLCPCB:C_0402
- removed J3: Display, Custom:OLED_1306_THT_pinheader
- removed R18, R19: 10kΩ, PCM_JLCPCB:R_0402
- moved D181 178.5 mm to (34.8, 221.2)
- moved D182 178.0 mm to (34.8, 223.2), turned to 180 degrees
- moved D191 177.8 mm to (59.8, 225.9), turned to -170 degrees
- moved D192 175.1 mm to (62.6, 226.1), turned to 160 degrees
- moved D183 174.8 mm to (37.8, 223.2), turned to 180 degrees
- moved D194 174.4 mm to (65.0, 230.8), turned to 90 degrees
- moved D193 173.9 mm to (65.0, 227.8), turned to 90 degrees
- moved D195 171.6 mm to (67.0, 230.8), turned to -90 degrees
- moved D184 171.5 mm to (40.8, 223.2), turned to 180 degrees
- moved D185 168.7 mm to (43.7, 223.7), turned to 160 degrees
- moved D186 167.1 mm to (46.3, 225.1), turned to 140 degrees
- moved D196 166.2 mm to (67.0, 227.8), turned to -90 degrees
- moved D187 165.9 mm to (48.6, 227.1), turned to 140 degrees
- moved D188 164.2 mm to (51.4, 228.4), turned to 170 degrees
- moved D161 163.6 mm to (29.1, 205.9), turned to -170 degrees
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Connections:
- U1 pad 4: /DISPLAY_SDA -> unconnected-(U1-GPIO0/XTAL_32K_P-Pad4)
- U1 pad 5: /DISPLAY_SCL -> unconnected-(U1-GPIO1/XTAL_32K_N-Pad5)
Routing:
- net +5V: track 58.0 -> 536.9 mm, vias 5 -> 93
- net Net-(C1-Pad2): track 202.8 -> 311.7 mm
- net /DISPLAY_SDA: track 100.8 -> 0.00 mm, vias 3 -> 0
- net /DISPLAY_SCL: track 98.1 -> 0.00 mm, vias 3 -> 0
- net /USB_D+: track 97.9 -> 29.4 mm
- net Net-(D156-DOUT): track 0.00 -> 32.5 mm, vias 0 -> 2
- net Net-(D123-DOUT): track 0.00 -> 31.4 mm, vias 0 -> 2
- net +3V3: track 238.5 -> 208.9 mm, vias 11 -> 10
- net /Leds/LED_DATA_5V: track 43.2 -> 21.0 mm
- net /USB_D-: track 100.3 -> 86.4 mm
- net Net-(D160-DOUT): track 0.00 -> 8.89 mm, vias 0 -> 2
- net Net-(D168-DOUT): track 0.00 -> 4.69 mm, vias 0 -> 2
- net GND: track 13.3 -> 17.8 mm, vias 55 -> 58
- net Net-(D197-DOUT): track 0.00 -> 3.99 mm
- net Net-(D129-DOUT): track 0.00 -> 3.87 mm
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Other:
- board size 112.5 x 109.8 mm -> 112.5 x 219.5 mm
- board text removed: "This might be the wrong footprint (maybe not)"
