File: pcb/fin-ltm.kicad_pcb (KiCad board)
At the start: 2 copper layers, 112.5 x 219.5 mm, 348 parts, among them J1 Connector, USB-TYPE-C-16P, J2 Test Connector, Q1 MMBT3904, Q2 HL3415A, U1 ESP32-C3FH4, U2 RT9080, U3 SN74LV1T34DBV, X1 40MHz, 15pF

Commit message: smaller tweaks
Parts:
- removed D163: WS2812B, PCM_JLCPCB:LED-SMD_4P-L1.6-W1.5_XL-1615RGBC-WS2812B
- added REF**: Station Box NT, Custom:Station Box NT, F.Cu at (100.4, 191.8)
- added REF**: Station Box NT, Custom:Station Box NT, F.Cu at (37.7, 204.1)
- moved D160 1.14 mm to (34.4, 203.2), turned to 135 degrees
- moved D157 0.79 mm to (27.2, 198.6)
- moved REF** 0.79 mm to (27.2, 198.6)
- moved D161 0.59 mm to (29.1, 205.8)
- moved D162 0.59 mm to (32.2, 205.5)
- moved REF** 0.59 mm to (29.1, 205.8)
- moved D158 0.52 mm to (30.3, 199.0), turned to 165 degrees
- moved D159 0.38 mm to (32.8, 200.9), turned to -60 degrees
- moved D164 0.16 mm to (37.7, 204.1), turned to -160 degrees
Connections:
- D164 pad 4: Net-(D163-DOUT) -> Net-(D162-DOUT)
Routing:
- net Net-(D160-DOUT): track 8.92 -> 0.00 mm
- net Net-(D157-DOUT): track 2.06 -> 0.00 mm
- net Net-(D161-DOUT): track 1.93 -> 0.11 mm
- net Net-(D162-DOUT): track 1.92 -> 0.11 mm
- net Net-(D158-DOUT): track 1.74 -> 0.00 mm
- net Net-(D159-DOUT): track 1.68 -> 0.00 mm

Commit message: finished led placement
Parts:
- removed D179, D181, D182, D203, D214, D215: WS2812B, PCM_JLCPCB:LED-SMD_4P-L1.6-W1.5_XL-1615RGBC-WS2812B
- added REF**: Station Box NB, Custom:Station Box NB, F.Cu at (35.0, 221.2)
- added REF**: Station Box NRV, Custom:Station Box NRV, F.Cu at (86.0, 219.8)
- added REF**: Station Box NLV, Custom:Station Box NLV, F.Cu at (61.7, 215.6)
- added REF**: Station Box NRV, Custom:Station Box NRV, F.Cu at (67.0, 220.5)
- added REF**: Station Box NT, Custom:Station Box NT, F.Cu at (82.8, 211.8)
- added REF**: Station Box NLV, Custom:Station Box NLV, F.Cu at (48.0, 212.5)
- added REF**: Station Box NLV, Custom:Station Box NLV, F.Cu at (43.0, 216.2)
- added REF**: Station Box NT, Custom:Station Box NT, F.Cu at (72.0, 211.8)
- added REF**: Station Box NRV, Custom:Station Box NRV, F.Cu at (67.0, 230.2)
- added REF**: Station Box NLV, Custom:Station Box NLV, F.Cu at (55.9, 211.2)
- added REF**: Station Box NT, Custom:Station Box NT, F.Cu at (44.1, 223.3)
- added REF**: Station Box NRV, Custom:Station Box NRV, F.Cu at (67.0, 227.2)
- added REF**: Station Box NRV, Custom:Station Box NRV, F.Cu at (51.9, 206.7)
- added REF**: Station Box NB, Custom:Station Box NB, F.Cu at (38.0, 221.2)
- moved D212 10.3 mm to (75.0, 211.8), turned to 180 degrees
- moved D337 4.00 mm to (84.8, 214.0)
- moved D338 4.00 mm to (85.0, 217.0)
- moved D339 4.00 mm to (86.0, 219.8)
- moved D213 3.00 mm to (78.0, 211.8)
- moved D206 2.87 mm to (61.5, 212.8), turned to -140 degrees
- moved D299 2.83 mm to (83.6, 179.8), turned to 60 degrees
- moved D180 2.82 mm to (35.0, 221.2), turned to 180 degrees
- moved D298 2.78 mm to (85.2, 177.5), turned to 50 degrees
- moved D210 2.27 mm to (68.4, 214.7), turned to 70 degrees
- moved D183 2.02 mm to (38.0, 221.2)
- moved D211 2.00 mm to (67.4, 217.5), turned to 70 degrees
- moved D207 1.74 mm to (64.5, 211.8), turned to 180 degrees
- moved D178 1.72 mm to (41.2, 218.8)
- moved D184 1.63 mm to (41.6, 221.8), turned to 160 degrees
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Connections:
- D180 pad 4: Net-(D179-DOUT) -> Net-(D178-DOUT)
- D183 pad 4: Net-(D182-DOUT) -> Net-(D180-DOUT)
- D204 pad 4: Net-(D203-DOUT) -> Net-(D202-DOUT)
- D216 pad 4: Net-(D215-DOUT) -> Net-(D213-DOUT)
Routing:
- net +5V: track 561.1 -> 1095.9 mm, vias 68 -> 225
- net GND: track 17.4 -> 67.0 mm, vias 59 -> 72
- net /Leds/LED_DATA_5V: track 36.5 -> 61.9 mm, vias 3 -> 4
- net Net-(D211-DOUT): track 0.00 -> 10.5 mm, vias 0 -> 2
- net Net-(D259-DOUT): track 0.00 -> 7.52 mm
- net Net-(D205-DOUT): track 0.00 -> 7.39 mm, vias 0 -> 2
- net Net-(D178-DOUT): track 0.00 -> 6.91 mm
- net Net-(D160-DOUT): track 0.00 -> 6.87 mm
- net Net-(D299-DOUT): track 0.00 -> 6.68 mm, vias 0 -> 2
- net Net-(D238-DOUT): track 0.00 -> 4.75 mm
- net Net-(D225-DOUT): track 0.00 -> 4.70 mm
- net Net-(D151-DOUT): track 0.00 -> 4.63 mm
- net Net-(D162-DOUT): track 0.11 -> 4.69 mm
- net Net-(D209-DOUT): track 0.00 -> 4.51 mm
- net Net-(D200-DOUT): track 0.00 -> 4.12 mm
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