File: pcb/leds.kicad_sch (KiCad schematic)
At the start: 235 parts

Commit message: Changing the silkscreen and changing led layout
Parts:
- removed D142, D171, D231, D246, D298, D300, D332: WS2812B, PCM_JLCPCB:LED-SMD_4P-L1.6-W1.5_XL-1615RGBC-WS2812B, symbol PCM_JLCPCB-Extended:LED, WS2812B, 1615
Connections:
- net at D141.1 (DOUT): now also D143.4 (DIN)
- net at D301.4 (DIN): now also D299.1 (DOUT)
- net at D172.4 (DIN): now also D170.1 (DOUT)
- net at D299.4 (DIN): now also D297.1 (DOUT)
- net at D230.1 (DOUT): now also D232.4 (DIN)
- net at D333.4 (DIN): now also D331.1 (DOUT)
- net at D245.1 (DOUT): now also D247.4 (DIN)

Commit message: smol tweak
Parts:
- removed D232, D247, D256: WS2812B, PCM_JLCPCB:LED-SMD_4P-L1.6-W1.5_XL-1615RGBC-WS2812B, symbol PCM_JLCPCB-Extended:LED, WS2812B, 1615
Connections:
- net at D230.1 (DOUT): now also D233.4 (DIN)
- net at D255.1 (DOUT): now also D257.4 (DIN)
- net at D245.1 (DOUT): now also D248.4 (DIN)

Commit message: tweaked layout
Parts:
- removed D226: WS2812B, PCM_JLCPCB:LED-SMD_4P-L1.6-W1.5_XL-1615RGBC-WS2812B, symbol PCM_JLCPCB-Extended:LED, WS2812B, 1615
- added D246, D256, D298: WS2812B, PCM_JLCPCB:LED-SMD_4P-L1.6-W1.5_XL-1615RGBC-WS2812B, symbol PCM_JLCPCB-Extended:LED, WS2812B, 1615
Connections:
- net +5V: now also D246.2 (VDD), D256.2 (VDD), D298.2 (VDD)
- net GND: now also D246.3 (GND), D256.3 (GND), D298.3 (GND)
- net at D225.1 (DOUT): now also D227.4 (DIN)
- net at D299.4 (DIN): now also D298.1 (DOUT); no longer D297.1 (DOUT)
- net at D230.1 (DOUT): now also D246.4 (DIN); no longer D233.4 (DIN)
- net at D257.4 (DIN): now also D256.1 (DOUT); no longer D255.1 (DOUT)
- new net: D297.1 (DOUT), D298.4 (DIN)
- new net: D255.1 (DOUT), D256.4 (DIN)
- new net: D233.4 (DIN), D246.1 (DOUT)

Commit message: smaller tweaks
Parts:
- removed D163: WS2812B, PCM_JLCPCB:LED-SMD_4P-L1.6-W1.5_XL-1615RGBC-WS2812B, symbol PCM_JLCPCB-Extended:LED, WS2812B, 1615
Connections:
- net at D164.4 (DIN): now also D162.1 (DOUT)

Commit message: finished led placement
Parts:
- removed D179, D181, D182, D203, D214, D215: WS2812B, PCM_JLCPCB:LED-SMD_4P-L1.6-W1.5_XL-1615RGBC-WS2812B, symbol PCM_JLCPCB-Extended:LED, WS2812B, 1615
Connections:
- net at D180.1 (DOUT): now also D183.4 (DIN)
- net at D180.4 (DIN): now also D178.1 (DOUT)
- net at D216.4 (DIN): now also D213.1 (DOUT)
- net at D204.4 (DIN): now also D202.1 (DOUT)

Commit message: linking leds to stations
Parts:
- renumbered D101 to D100, D102 to D101, D103 to D102, D104 to D103, D105 to D104, D106 to D105, D107 to D106, D108 to D107, D109 to D108, D110 to D109, D111 to D110, D112 to D111, D113 to D112, D114 to D113, D115 to D114, D116 to D115, D117 to D116, D118 to D117, D119 to D118, D120 to D119, D121 to D120, D122 to D121, D123 to D122, D124 to D123, D125 to D124, D126 to D125, D127 to D126, D129 to D127, D130 to D128, D131 to D129, D132 to D130, D133 to D131, D134 to D132, D135 to D133, D136 to D134, D138 to D135, D139 to D136, D140 to D137, D141 to D138, D143 to D139, D144 to D140, D145 to D141, D146 to D142, D147 to D143, D148 to D144, D149 to D145, D150 to D146, D151 to D147, D152 to D148, D153 to D149, D154 to D150, D155 to D151, D156 to D152, D157 to D153, D158 to D154, D159 to D155, D160 to D156, D161 to D157, D162 to D158, D164 to D159, D165 to D160, D166 to D161, D167 to D162, D168 to D163, D169 to D164, D170 to D165, D172 to D166, D173 to D167, D174 to D168, D175 to D169, D176 to D170, D177 to D171, D178 to D172, D180 to D173, D183 to D174, D184 to D175, D185 to D176, D186 to D177, D187 to D178, D188 to D179, D189 to D180, D190 to D181, D191 to D182, D192 to D183, D193 to D184, D194 to D185, D195 to D186, D196 to D187, D197 to D188, D198 to D189, D199 to D190, D200 to D191, D201 to D192, D202 to D193, D204 to D194, D205 to D195, D206 to D196, D207 to D197, D208 to D198, D209 to D199, D210 to D200, D211 to D201, D212 to D202, D213 to D203, D216 to D204, D217 to D205, D218 to D206, D219 to D207, D220 to D208, D221 to D209, D222 to D210, D223 to D211, D224 to D212, D225 to D213, D227 to D214, D228 to D215, D229 to D216, D230 to D217, D246 to D218, D233 to D219, D234 to D220, D235 to D221, D236 to D222, D237 to D223, D238 to D224, D239 to D225, D240 to D226, D241 to D227, D242 to D228, D243 to D229, D244 to D230, D245 to D231, D248 to D232, D249 to D233, D250 to D234, D251 to D235, D252 to D236, D253 to D237, D254 to D238, D255 to D239, D256 to D240, D257 to D241, D258 to D242, D259 to D243, D260 to D244, D261 to D245, D262 to D246, D263 to D247, D264 to D248, D265 to D249, D266 to D250, D267 to D251, D269 to D252, D270 to D253, D271 to D254, D272 to D255, D273 to D256, D274 to D257, D275 to D258, D276 to D259, D277 to D260, D278 to D261, D279 to D262, D280 to D263, D281 to D264, D282 to D265, D283 to D266, D284 to D267, D285 to D268, D286 to D269, D288 to D270, D289 to D271, D290 to D272, D291 to D273, D292 to D274, D293 to D275, D294 to D276, D295 to D277, D296 to D278, D297 to D279, D298 to D280, D299 to D281, D301 to D282, D302 to D283, D303 to D284, D304 to D285, D305 to D286, D306 to D287, D307 to D288, D308 to D289, D309 to D290, D310 to D291, D311 to D292, D312 to D293, D313 to D294, D314 to D295, D315 to D296, D316 to D297, D317 to D298, D318 to D299, D319 to D300, D320 to D301, D321 to D302, D322 to D303, D323 to D304, D324 to D305, D325 to D306, D326 to D307, D327 to D308, D328 to D309, D329 to D310, D330 to D311, D331 to D312, D333 to D313, D334 to D314, D335 to D315, D336 to D316, D337 to D317, D338 to D318, D339 to D319

Commit message: added led decoupling caps
Parts:
- added C100, C101, C102, C103, C104, C105, C106, C107, C108, C109, C110, C111, C112, C113, C114, C115, C116, C117, C118, C119, C120, C121, C122, C123, C124, C125, C126, C127, C128, C129, C130, C131, C132, C133, C134, C135, C136, C137, C138, C139: 10uF, PCM_JLCPCB:C_0402, symbol PCM_JLCPCB-Capacitors:0402,10uF
Connections:
- net +5V: now also C100.1, C101.1, C102.1, C103.1, C104.1, C105.1, C106.1, C107.1, C108.1, C109.1, C110.1, C111.1, C112.1, C113.1, C114.1, C115.1, C116.1, C117.1, C118.1, C119.1, C120.1, C121.1, C122.1, C123.1, C124.1, C125.1, C126.1, C127.1, C128.1, C129.1, C130.1, C131.1, C132.1, C133.1, C134.1, C135.1, C136.1, C137.1, C138.1, C139.1
- net GND: now also C100.2, C101.2, C102.2, C103.2, C104.2, C105.2, C106.2, C107.2, C108.2, C109.2, C110.2, C111.2, C112.2, C113.2, C114.2, C115.2, C116.2, C117.2, C118.2, C119.2, C120.2, C121.2, C122.2, C123.2, C124.2, C125.2, C126.2, C127.2, C128.2, C129.2, C130.2, C131.2, C132.2, C133.2, C134.2, C135.2, C136.2, C137.2, C138.2, C139.2

Commit message: pcb update
Parts:
- added D320: WS2812B, PCM_JLCPCB:LED-SMD_4P-L1.6-W1.5_XL-1615RGBC-WS2812B, symbol PCM_JLCPCB-Extended:LED, WS2812B, 1615
Connections:
- net +5V: now also D320.2 (VDD)
- net GND: now also D320.3 (GND)
- net at D188.4 (DIN): now also D320.1 (DOUT); no longer D187.1 (DOUT)
- new net: D187.1 (DOUT), D320.4 (DIN)
Other:
- moved on the sheet: D174, D175, D176, D177, D178, D179, D180, D181, D182, D183, D184, D185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
