File: pcb/leds.kicad_sch (KiCad schematic)
At the start: 261 parts

Commit message: wrote more definitions
Parts:
- renumbered D320 to D188, D188 to D189, D189 to D190, D190 to D191, D191 to D192, D192 to D193, D193 to D194, D194 to D195, D195 to D196, D196 to D197, D197 to D198, D198 to D199, D199 to D200, D200 to D201, D201 to D202, D202 to D203, D203 to D204, D204 to D205, D205 to D206, D206 to D207, D207 to D208, D208 to D209, D209 to D210, D210 to D211, D211 to D212, D212 to D213, D213 to D214, D214 to D215, D215 to D216, D216 to D217, D217 to D218, D218 to D219, D219 to D220, D220 to D221, D221 to D222, D222 to D223, D223 to D224, D224 to D225, D225 to D226, D226 to D227, D227 to D228, D228 to D229, D229 to D230, D230 to D231, D231 to D232, D232 to D233, D233 to D234, D234 to D235, D235 to D236, D236 to D237, D237 to D238, D238 to D239, D239 to D240, D240 to D241, D241 to D242, D242 to D243, D243 to D244, D244 to D245, D245 to D246, D246 to D247, D247 to D248, D248 to D249, D249 to D250, D250 to D251, D251 to D252, D252 to D253, D253 to D254, D254 to D255, D255 to D256, D256 to D257, D257 to D258, D258 to D259, D259 to D260, D260 to D261, D261 to D262, D262 to D263, D263 to D264, D264 to D265, D265 to D266, D266 to D267, D267 to D268, D268 to D269, D269 to D270, D270 to D271, D271 to D272, D272 to D273, D273 to D274, D274 to D275, D275 to D276, D276 to D277, D277 to D278, D278 to D279, D279 to D280, D280 to D281, D281 to D282, D282 to D283, D283 to D284, D284 to D285, D285 to D286, D286 to D287, D287 to D288, D288 to D289, D289 to D290, D290 to D291, D291 to D292, D292 to D293, D293 to D294, D294 to D295, D295 to D296, D296 to D297, D297 to D298, D298 to D299, D299 to D300, D300 to D301, D301 to D302, D302 to D303, D303 to D304, D304 to D305, D305 to D306, D306 to D307, D307 to D308, D308 to D309, D309 to D310, D310 to D311, D311 to D312, D312 to D313, D313 to D314, D314 to D315, D315 to D316, D316 to D317, D317 to D318, D318 to D319, D319 to D320

Commit message: added haaparanta
Parts:
- added D321, D322: WS2812B, PCM_JLCPCB:LED-SMD_4P-L1.6-W1.5_XL-1615RGBC-WS2812B, symbol PCM_JLCPCB-Extended:LED, WS2812B, 1615
Connections:
- net +5V: now also D321.2 (VDD), D322.2 (VDD)
- net GND: now also D321.3 (GND), D322.3 (GND)
- net at D109.1 (DOUT): now also D321.4 (DIN); no longer D110.4 (DIN)
- new net: D321.1 (DOUT), D322.4 (DIN)
- new net: D110.4 (DIN), D322.1 (DOUT)
