File: pcb/fin-ltm.kicad_sch (KiCad schematic)
At the start: 64 parts, among them J1 Connector, USB-TYPE-C-16P, J2 Test Connector, Q1 HL3415A, Q2 MMBT3904, U1 RT9080, U2 ESP32-C3FH4, U3 SN74LV1T34DBV, X1 40MHz, 15pF

Commit message: capcitor fix
Parts:
- C10, C12, C20, C21, C5: footprint PCM_JLCPCB:C_0603 -> PCM_JLCPCB:C_0402; symbol PCM_JLCPCB-Capacitors:0603,10uF -> PCM_JLCPCB-Capacitors:0402,10uF; LCSC C19702 -> C15525; Part CL10A106KP8NNNC -> CL05A106MQ5NUNC; Stock 9881407 -> 3940889; Tolerance ±10% -> ±20%; Voltage Rated 10V -> 6.3V
Changed lines of the file:
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@@
 	)
 	(symbol
-		(lib_id "PCM_JLCPCB-Capacitors:0603,10uF")
+		(lib_id "PCM_JLCPCB-Capacitors:0402,10uF")
 		(at 154.94 175.26 0)
 		(unit 1)
@@
 			)
 		)
-		(property "Footprint" "PCM_JLCPCB:C_0603"
+		(property "Footprint" "PCM_JLCPCB:C_0402"
 			(at 153.162 175.26 90)
 			(hide yes)
@@
 			)
 		)
-		(property "Datasheet" "https://www.lcsc.com/datasheet/lcsc_datasheet_2304140030_Samsung-Electro-Mechanics-CL10A106KP8NNNC_C19702.pdf"
+		(property "Datasheet" "https://www.lcsc.com/datasheet/lcsc_datasheet_2208231630_Samsung-Electro-Mechanics-CL05A106MQ5NUNC_C15525.pdf"
 			(at 154.94 175.26 0)
 			(hide yes)
@@
 			)
 		)
-		(property "Description" "10V 10uF X5R ±10% 0603 Multilayer Ceramic Capacitors MLCC - SMD/SMT ROHS"
+		(property "Description" "6.3V 10uF X5R ±20% 0402 Multilayer Ceramic Capacitors MLCC - SMD/SMT ROHS"
 			(at 154.94 175.26 0)
 			(hide yes)
@@
 			)
 		)
-		(property "LCSC" "C19702"
+		(property "LCSC" "C15525"
 			(at 154.94 175.26 0)
 			(hide yes)
@@
 			)
 		)
-		(property "Stock" "9881407"
+		(property "Stock" "3940889"
 			(at 154.94 175.26 0)
 			(hide yes)
@@
 			)
 		)
-		(property "Part" "CL10A106KP8NNNC"
+		(property "Part" "CL05A106MQ5NUNC"
 			(at 154.94 175.26 0)
 			(hide yes)
@@
 			)
 		)
-		(property "Voltage Rated" "10V"
+		(property "Voltage Rated" "6.3V"
 			(at 157.48 177.8 0)
 			(show_name no)
@@
 			)
 		)
-		(property "Tolerance" "±10%"
+		(property "Tolerance" "±20%"
 			(at 154.94 175.26 0)
 			(hide yes)
@@
 	)
 	(symbol
-		(lib_id "PCM_JLCPCB-Capacitors:0603,10uF")
+		(lib_id "PCM_JLCPCB-Capacitors:0402,10uF")
 		(at 163.83 175.26 0)
 		(unit 1)
@@
 			)
 		)
-		(property "Footprint" "PCM_JLCPCB:C_0603"
+		(property "Footprint" "PCM_JLCPCB:C_0402"
 			(at 162.052 175.26 90)
 			(hide yes)
@@
 			)
 		)
-		(property "Datasheet" "https://www.lcsc.com/datasheet/lcsc_datasheet_2304140030_Samsung-Electro-Mechanics-CL10A106KP8NNNC_C19702.pdf"
+		(property "Datasheet" "https://www.lcsc.com/datasheet/lcsc_datasheet_2208231630_Samsung-Electro-Mechanics-CL05A106MQ5NUNC_C15525.pdf"
 			(at 163.83 175.26 0)
 			(hide yes)
@@
 			)
 		)
-		(property "Description" "10V 10uF X5R ±10% 0603 Multilayer Ceramic Capacitors MLCC - SMD/SMT ROHS"
+		(property "Description" "6.3V 10uF X5R ±20% 0402 Multilayer Ceramic Capacitors MLCC - SMD/SMT ROHS"
 			(at 163.83 175.26 0)
 			(hide yes)
@@
 			)
 		)
-		(property "LCSC" "C19702"
+		(property "LCSC" "C15525"
 			(at 163.83 175.26 0)
 			(hide yes)
@@
 			)
 		)
-		(property "Stock" "9881407"
+		(property "Stock" "3940889"
 			(at 163.83 175.26 0)
 			(hide yes)
@@
 			)
 		)
-		(property "Part" "CL10A106KP8NNNC"
+		(property "Part" "CL05A106MQ5NUNC"
 			(at 163.83 175.26 0)
 			(hide yes)
@@
 			)
 		)
-		(property "Voltage Rated" "10V"
+		(property "Voltage Rated" "6.3V"
 			(at 166.37 177.8 0)
 			(show_name no)
@@
 			)
 		)
-		(property "Tolerance" "±10%"
+		(property "Tolerance" "±20%"
 			(at 163.83 175.26 0)
 			(hide yes)
@@
 	)
 	(symbol
-		(lib_id "PCM_JLCPCB-Capacitors:0603,10uF")
+		(lib_id "PCM_JLCPCB-Capacitors:0402,10uF")
 		(at 81.28 46.99 0)
 		(unit 1)
@@
 			)
 		)
-		(property "Footprint" "PCM_JLCPCB:C_0603"
+		(property "Footprint" "PCM_JLCPCB:C_0402"
 			(at 79.502 46.99 90)
 			(hide yes)
@@
 			)
 		)
-		(property "Datasheet" "https://www.lcsc.com/datasheet/lcsc_datasheet_2304140030_Samsung-Electro-Mechanics-CL10A106KP8NNNC_C19702.pdf"
+		(property "Datasheet" "https://www.lcsc.com/datasheet/lcsc_datasheet_2208231630_Samsung-Electro-Mechanics-CL05A106MQ5NUNC_C15525.pdf"
 			(at 81.28 46.99 0)
 			(hide yes)
@@
 			)
 		)
-		(property "Description" "10V 10uF X5R ±10% 0603 Multilayer Ceramic Capacitors MLCC - SMD/SMT ROHS"
+		(property "Description" "6.3V 10uF X5R ±20% 0402 Multilayer Ceramic Capacitors MLCC - SMD/SMT ROHS"
 			(at 81.28 46.99 0)
 			(hide yes)
@@
 			)
 		)
-		(property "LCSC" "C19702"
+		(property "LCSC" "C15525"
 			(at 81.28 46.99 0)
 			(hide yes)
@@
 			)
 		)
-		(property "Stock" "9881407"
+		(property "Stock" "3940889"
 			(at 81.28 46.99 0)
 			(hide yes)
@@
 			)
 		)
-		(property "Part" "CL10A106KP8NNNC"
+		(property "Part" "CL05A106MQ5NUNC"
 			(at 81.28 46.99 0)
 			(hide yes)
@@
 			)
 		)
-		(property "Voltage Rated" "10V"
+		(property "Voltage Rated" "6.3V"
 			(at 83.312 49.0362 0)
 			(show_name no)
@@
 			)
 		)
-		(property "Tolerance" "±10%"
+		(property "Tolerance" "±20%"
 			(at 81.28 46.99 0)
 			(hide yes)
@@
 	)
 	(symbol
-		(lib_id "PCM_JLCPCB-Capacitors:0603,10uF")
+		(lib_id "PCM_JLCPCB-Capacitors:0402,10uF")
 		(at 44.45 39.37 0)
 		(unit 1)
@@
 			)
 		)
-		(property "Footprint" "PCM_JLCPCB:C_0603"
+		(property "Footprint" "PCM_JLCPCB:C_0402"
 			(at 42.672 39.37 90)
 			(hide yes)
@@
 			)
 		)
-		(property "Datasheet" "https://www.lcsc.com/datasheet/lcsc_datasheet_2304140030_Samsung-Electro-Mechanics-CL10A106KP8NNNC_C19702.pdf"
+		(property "Datasheet" "https://www.lcsc.com/datasheet/lcsc_datasheet_2208231630_Samsung-Electro-Mechanics-CL05A106MQ5NUNC_C15525.pdf"
 			(at 44.45 39.37 0)
 			(hide yes)
@@
 			)
 		)
-		(property "Description" "10V 10uF X5R ±10% 0603 Multilayer Ceramic Capacitors MLCC - SMD/SMT ROHS"
+		(property "Description" "6.3V 10uF X5R ±20% 0402 Multilayer Ceramic Capacitors MLCC - SMD/SMT ROHS"
 			(at 44.45 39.37 0)
 			(hide yes)
@@
 			)
 		)
-		(property "LCSC" "C19702"
+		(property "LCSC" "C15525"
 			(at 44.45 39.37 0)
 			(hide yes)
@@
 			)
 		)
-		(property "Stock" "9881407"
+		(property "Stock" "3940889"
 			(at 44.45 39.37 0)
 			(hide yes)
@@
 			)
 		)
-		(property "Part" "CL10A106KP8NNNC"
+		(property "Part" "CL05A106MQ5NUNC"
 			(at 44.45 39.37 0)
 			(hide yes)
@@
 			)
 		)
-		(property "Voltage Rated" "10V"
+		(property "Voltage Rated" "6.3V"
 			(at 46.482 41.4162 0)
 			(show_name no)
@@
 			)
 		)
-		(property "Tolerance" "±10%"
+		(property "Tolerance" "±20%"
 			(at 44.45 39.37 0)
 			(hide yes)
@@
 	)
 	(symbol
-		(lib_id "PCM_JLCPCB-Capacitors:0603,10uF")
+		(lib_id "PCM_JLCPCB-Capacitors:0402,10uF")
 		(at 121.92 66.04 0)
 		(unit 1)
@@
 			)
 		)
-		(property "Footprint" "PCM_JLCPCB:C_0603"
+		(property "Footprint" "PCM_JLCPCB:C_0402"
 			(at 120.142 66.04 90)
 			(hide yes)
@@
 			)
 		)
-		(property "Datasheet" "https://www.lcsc.com/datasheet/lcsc_datasheet_2304140030_Samsung-Electro-Mechanics-CL10A106KP8NNNC_C19702.pdf"
+		(property "Datasheet" "https://www.lcsc.com/datasheet/lcsc_datasheet_2208231630_Samsung-Electro-Mechanics-CL05A106MQ5NUNC_C15525.pdf"
 			(at 121.92 66.04 0)
 			(hide yes)
@@
 			)
 		)
-		(property "Description" "10V 10uF X5R ±10% 0603 Multilayer Ceramic Capacitors MLCC - SMD/SMT ROHS"
+		(property "Description" "6.3V 10uF X5R ±20% 0402 Multilayer Ceramic Capacitors MLCC - SMD/SMT ROHS"
 			(at 121.92 66.04 0)
 			(hide yes)
@@
 			)
 		)
-		(property "LCSC" "C19702"
+		(property "LCSC" "C15525"
 			(at 121.92 66.04 0)
 			(hide yes)
@@
 			)
 		)
-		(property "Stock" "9881407"
+		(property "Stock" "3940889"
 			(at 121.92 66.04 0)
 			(hide yes)
@@
 			)
 		)
-		(property "Part" "CL10A106KP8NNNC"
+		(property "Part" "CL05A106MQ5NUNC"
 			(at 121.92 66.04 0)
 			(hide yes)
@@
 			)
 		)
-		(property "Voltage Rated" "10V"
+		(property "Voltage Rated" "6.3V"
 			(at 124.46 68.58 0)
 			(show_name no)
@@
 			)
 		)
-		(property "Tolerance" "±10%"
+		(property "Tolerance" "±20%"
 			(at 121.92 66.04 0)
 			(hide yes)
