File: pcb/fin-ltm.kicad_sch (KiCad schematic)
At the start: 64 parts, among them J1 Connector, USB-TYPE-C-16P, J2 Test Connector, Q1 HL3415A, Q2 MMBT3904, U1 RT9080, U2 ESP32-C3FH4, U3 SN74LV1T34DBV, X1 40MHz, 15pF

Commit message: add debug pin
Connections:
- net +3V3: now also J2.8 (+3V3); no longer J2.7 (+3V3)
- net BRIGHTNESS_DOWN_BUTTON: now also J2.4 (Boot)
- net GND: now also J2.7 (GND); no longer J2.6 (GND)
- net MCU_RX: now also J2.5 (TX); no longer J2.4 (TX)
- net MCU_TX: now also J2.6 (RX); no longer J2.5 (RX)
Changed lines of the file:
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@@
 	)
 	(junction
+		(at 180.34 48.26)
+		(diameter 0)
+		(color 0 0 0 0)
+	)
+	(junction
 		(at 115.57 78.74)
 		(diameter 0)
@@
 	(wire
 		(pts
+			(xy 265.43 105.41) (xy 269.24 105.41)
+		)
+		(stroke
+			(width 0)
+			(type default)
+		)
+	)
+	(wire
+		(pts
 			(xy 50.8 43.18) (xy 54.61 43.18)
 		)
@@
 	(wire
 		(pts
-			(xy 266.7 104.14) (xy 269.24 104.14)
-		)
-		(stroke
-			(width 0)
-			(type default)
-		)
-	)
-	(wire
-		(pts
 			(xy 196.85 124.46) (xy 196.85 116.84)
 		)
@@
 	(wire
 		(pts
-			(xy 266.7 109.22) (xy 269.24 109.22)
+			(xy 265.43 110.49) (xy 269.24 110.49)
 		)
 		(stroke
@@
 	(wire
 		(pts
-			(xy 266.7 106.68) (xy 269.24 106.68)
+			(xy 265.43 107.95) (xy 269.24 107.95)
 		)
 		(stroke
@@
 	(wire
 		(pts
-			(xy 173.99 48.26) (xy 208.28 48.26)
+			(xy 173.99 48.26) (xy 180.34 48.26)
 		)
 		(stroke
@@
 	(wire
 		(pts
+			(xy 180.34 48.26) (xy 208.28 48.26)
+		)
+		(stroke
+			(width 0)
+			(type default)
+		)
+	)
+	(wire
+		(pts
+			(xy 265.43 102.87) (xy 269.24 102.87)
+		)
+		(stroke
+			(width 0)
+			(type default)
+		)
+	)
+	(wire
+		(pts
 			(xy 236.22 34.29) (xy 236.22 35.56)
 		)
@@
 	(wire
 		(pts
+			(xy 180.34 33.02) (xy 180.34 48.26)
+		)
+		(stroke
+			(width 0)
+			(type default)
+		)
+	)
+	(wire
+		(pts
 			(xy 64.77 48.26) (xy 64.77 53.34)
 		)
@@
 	(wire
 		(pts
+			(xy 176.53 33.02) (xy 180.34 33.02)
+		)
+		(stroke
+			(width 0)
+			(type default)
+		)
+	)
+	(wire
+		(pts
 			(xy 86.36 43.18) (xy 90.17 43.18)
 		)
@@
 	)
 	(label "Reset"
-		(at 266.7 104.14 180)
+		(at 265.43 102.87 180)
 		(effects
 			(font
@@
 	)
 	(label "MCU_TX"
-		(at 266.7 109.22 180)
+		(at 265.43 110.49 180)
 		(effects
 			(font
@@
 		)
 	)
+	(label "Boot"
+		(at 265.43 105.41 180)
+		(effects
+			(font
+				(size 1.27 1.27)
+			)
+			(justify right bottom)
+		)
+	)
 	(label "MCU_RX"
 		(at 200.66 63.5 180)
@@
 	)
 	(label "MCU_RX"
-		(at 266.7 106.68 180)
+		(at 265.43 107.95 180)
 		(effects
 			(font
@@
 		)
 	)
+	(label "Boot"
+		(at 176.53 33.02 0)
+		(effects
+			(font
+				(size 1.27 1.27)
+			)
+			(justify left bottom)
+		)
+	)
 	(label "USB_D-"
 		(at 41.91 55.88 0)
@@
 	(symbol
 		(lib_id "power:GND")
-		(at 269.24 111.76 270)
+		(at 269.24 113.03 270)
 		(unit 1)
 		(body_style 1)
@@
 		(fields_autoplaced yes)
 		(property "Reference" "#PWR048"
-			(at 262.89 111.76 0)
+			(at 262.89 113.03 0)
 			(hide yes)
 			(show_name no)
@@
 		)
 		(property "Value" "GND"
-			(at 265.43 111.7599 90)
+			(at 265.43 113.0299 90)
 			(show_name no)
 			(do_not_autoplace no)
@@
 		)
 		(property "Footprint" ""
-			(at 269.24 111.76 0)
+			(at 269.24 113.03 0)
 			(hide yes)
 			(show_name no)
@@
 		)
 		(property "Datasheet" ""
-			(at 269.24 111.76 0)
+			(at 269.24 113.03 0)
 			(hide yes)
 			(show_name no)
@@
 		)
 		(property "Description" "Power symbol creates a global label with name \"GND\" , ground"
-			(at 269.24 111.76 0)
+			(at 269.24 113.03 0)
 			(hide yes)
 			(show_name no)
@@
 		(pin "7"
 		)
+		(pin "8"
+		)
 		(instances
 			(project "fin-ltm"
@@
 	(symbol
 		(lib_id "power:GND")
-		(at 269.24 101.6 270)
+		(at 269.24 100.33 270)
 		(unit 1)
 		(body_style 1)
@@
 		(fields_autoplaced yes)
 		(property "Reference" "#PWR046"
-			(at 262.89 101.6 0)
+			(at 262.89 100.33 0)
 			(hide yes)
 			(show_name no)
@@
 		)
 		(property "Value" "GND"
-			(at 265.43 101.5999 90)
+			(at 265.43 100.3299 90)
 			(show_name no)
 			(do_not_autoplace no)
@@
 		)
 		(property "Footprint" ""
-			(at 269.24 101.6 0)
+			(at 269.24 100.33 0)
 			(hide yes)
 			(show_name no)
@@
 		)
 		(property "Datasheet" ""
-			(at 269.24 101.6 0)
+			(at 269.24 100.33 0)
 			(hide yes)
 			(show_name no)
@@
 		)
 		(property "Description" "Power symbol creates a global label with name \"GND\" , ground"
-			(at 269.24 101.6 0)
+			(at 269.24 100.33 0)
 			(hide yes)
 			(show_name no)
@@
 	(symbol
 		(lib_id "power:+3V3")
-		(at 269.24 114.3 90)
+		(at 269.24 115.57 90)
 		(unit 1)
 		(body_style 1)
@@
 		(fields_autoplaced yes)
 		(property "Reference" "#PWR049"
-			(at 273.05 114.3 0)
+			(at 273.05 115.57 0)
 			(hide yes)
 			(show_name no)
@@
 		)
 		(property "Value" "+3V3"
-			(at 265.43 114.2999 90)
+			(at 265.43 115.5699 90)
 			(show_name no)
 			(do_not_autoplace no)
@@
 		)
 		(property "Footprint" ""
-			(at 269.24 114.3 0)
+			(at 269.24 115.57 0)
 			(hide yes)
 			(show_name no)
@@
 		)
 		(property "Datasheet" ""
-			(at 269.24 114.3 0)
+			(at 269.24 115.57 0)
 			(hide yes)
 			(show_name no)
@@
 		)
 		(property "Description" "Power symbol creates a global label with name \"+3V3\""
-			(at 269.24 114.3 0)
+			(at 269.24 115.57 0)
 			(hide yes)
 			(show_name no)
@@
 	(symbol
 		(lib_id "power:+5V")
-		(at 269.24 99.06 90)
+		(at 269.24 97.79 90)
 		(unit 1)
 		(body_style 1)
@@
 		(fields_autoplaced yes)
 		(property "Reference" "#PWR045"
-			(at 273.05 99.06 0)
+			(at 273.05 97.79 0)
 			(hide yes)
 			(show_name no)
@@
 		)
 		(property "Value" "+5V"
-			(at 265.43 99.0599 90)
+			(at 265.43 97.7899 90)
 			(show_name no)
 			(do_not_autoplace no)
@@
 		)
 		(property "Footprint" ""
-			(at 269.24 99.06 0)
+			(at 269.24 97.79 0)
 			(hide yes)
 			(show_name no)
@@
 		)
 		(property "Datasheet" ""
-			(at 269.24 99.06 0)
+			(at 269.24 97.79 0)
 			(hide yes)
 			(show_name no)
@@
 		)
 		(property "Description" "Power symbol creates a global label with name \"+5V\""
-			(at 269.24 99.06 0)
+			(at 269.24 97.79 0)
 			(hide yes)
 			(show_name no)
